Commit message: added isaac sim integration

File: robots/common/franka_arm.ros2_control.xacro (robot description, xacro)
@@ -7,4 +7,6 @@
                  fake_sensor_commands:=false
                  gazebo:=false
+                 isaac:=false
+                 namespace:=franka_ns
                  hand:=false
                  gazebo_effort:=false
@@ -16,6 +18,6 @@
           <param name="arm_id">${arm_id}</param>
           <param name="prefix">${arm_prefix}</param>
-          <xacro:if value="${use_fake_hardware}">
-            <plugin>fake_components/GenericSystem</plugin>
+          <xacro:if value="${use_fake_hardware and isaac == 0}">
+            <plugin>mock_components/GenericSystem</plugin>
             <param name="fake_sensor_commands">${fake_sensor_commands}</param>
             <param name="state_following_offset">0.0</param>
@@ -23,4 +25,16 @@
           <xacro:if value="${gazebo}">
             <plugin>franka_ign_ros2_control/IgnitionSystem</plugin>
+          </xacro:if>
+          <!-- ADDITION FOR ISAAC SIM -->
+          <xacro:if value="${isaac}">
+            <plugin>topic_based_ros2_control/TopicBasedSystem</plugin>
+            <xacro:if value="${namespace == ''}">
+              <param name="joint_commands_topic">/isaac_joint_commands</param>
+              <param name="joint_states_topic">/isaac_joint_states</param>
+            </xacro:if>
+            <xacro:if value="${namespace != ''}">
+              <param name="joint_commands_topic">/${namespace}/isaac_joint_commands</param>
+              <param name="joint_states_topic">/${namespace}/isaac_joint_states</param>
+            </xacro:if>
           </xacro:if>
           <xacro:if value="${use_fake_hardware == 0 and gazebo == 0}">
@@ -46,7 +60,10 @@
             <param name="initial_value">${initial_position}</param>
           </state_interface>
-          <state_interface name="velocity"/>
+          <state_interface name="velocity">
             <param name="initial_value">0.0</param>
-          <state_interface name="effort"/>
+          </state_interface>
+          <state_interface name="effort">
+            <param name="initial value">0.0</param>
+          </state_interface>
         </joint>
       </xacro:macro>
@@ -61,28 +78,30 @@
         <xacro:configure_joint joint_name="${arm_id}_finger_joint1" initial_position="0.0" />
       </xacro:if>
-      <xacro:macro name="general_purpose_io" params="prefix command_interface index">
-        <gpio name="${prefix}">
-          <command_interface name="${command_interface}"/>
-          <param name="index">${index}</param>
-        </gpio>
-      </xacro:macro>
-      <!-- Cartesian velocity interfaces -->
-      <xacro:general_purpose_io prefix="vx" command_interface="cartesian_velocity" index="0"/>
-      <xacro:general_purpose_io prefix="vy" command_interface="cartesian_velocity" index="1"/>
-      <xacro:general_purpose_io prefix="vz" command_interface="cartesian_velocity" index="2"/>
-      <xacro:general_purpose_io prefix="wx" command_interface="cartesian_velocity" index="3"/>
-      <xacro:general_purpose_io prefix="wy" command_interface="cartesian_velocity" index="4"/>
-      <xacro:general_purpose_io prefix="wz" command_interface="cartesian_velocity" index="5"/>
-      <!-- Cartesian pose interfaces, in total 16 interfaces -->
-      <xacro:macro name="loop" params="i">
-        <xacro:unless value="${i == 16}">
-          <xacro:general_purpose_io prefix="${i}" command_interface="cartesian_pose_command" index="${i}"/>
-          <xacro:loop i="${i+1}"/>
-        </xacro:unless>
-      </xacro:macro>
-      <xacro:loop i="0"/>
-      <!-- Elbow command interfaces -->
-      <xacro:general_purpose_io prefix="joint_3_position" command_interface="elbow_command" index="0"/>
-      <xacro:general_purpose_io prefix="joint_4_sign" command_interface="elbow_command" index="1"/>
+      <xacro:unless value="${isaac}">
+        <xacro:macro name="general_purpose_io" params="prefix command_interface index">
+          <gpio name="${prefix}">
+            <command_interface name="${command_interface}"/>
+            <param name="index">${index}</param>
+          </gpio>
+        </xacro:macro>
+        <!-- Cartesian velocity interfaces -->
+        <xacro:general_purpose_io prefix="vx" command_interface="cartesian_velocity" index="0"/>
+        <xacro:general_purpose_io prefix="vy" command_interface="cartesian_velocity" index="1"/>
+        <xacro:general_purpose_io prefix="vz" command_interface="cartesian_velocity" index="2"/>
+        <xacro:general_purpose_io prefix="wx" command_interface="cartesian_velocity" index="3"/>
+        <xacro:general_purpose_io prefix="wy" command_interface="cartesian_velocity" index="4"/>
+        <xacro:general_purpose_io prefix="wz" command_interface="cartesian_velocity" index="5"/>
+        <!-- Cartesian pose interfaces, in total 16 interfaces -->
+        <xacro:macro name="loop" params="i">
+          <xacro:unless value="${i == 16}">
+            <xacro:general_purpose_io prefix="${i}" command_interface="cartesian_pose_command" index="${i}"/>
+            <xacro:loop i="${i+1}"/>
+          </xacro:unless>
+        </xacro:macro>
+        <xacro:loop i="0"/>
+        <!-- Elbow command interfaces -->
+        <xacro:general_purpose_io prefix="joint_3_position" command_interface="elbow_command" index="0"/>
+        <xacro:general_purpose_io prefix="joint_4_sign" command_interface="elbow_command" index="1"/>
+      </xacro:unless>
     </ros2_control>
     <xacro:if value="${gazebo}">

File: robots/common/franka_robot.xacro (robot description, xacro)
@@ -19,4 +19,6 @@
                       special_connection:=''
                       gazebo:='false'
+                      isaac:='false'
+                      namespace:=''
                       with_sc:='false'
                       ros2_control:=false
@@ -149,4 +151,6 @@
           fake_sensor_commands="${fake_sensor_commands}"
           gazebo="${gazebo}"
+          isaac="${isaac}"
+          namespace="${namespace}"
           hand="${hand}"
           gazebo_effort="${gazebo_effort}"

File: robots/fr3/fr3.urdf.xacro (robot description, xacro)
@@ -40,4 +40,6 @@
   <!-- Should the robot be spawned in Gazebo?" -->
   <xacro:arg name="gazebo" default="false" />
+  <!-- Enable Topic Based ROS2 Control communication with Isaac Sim? -->
+  <xacro:arg name="isaac" default="false" />
   <!-- Should the robot be spawned in Gazebo with effort interfaces?" -->
   <xacro:arg name="gazebo_effort" default="false" />
@@ -53,4 +55,5 @@
                       dynamics="${xacro.load_yaml('$(find franka_description)/robots/fr3/dynamics.yaml')}"
                       gazebo="$(arg gazebo)"
+                      isaac="$(arg isaac)"
                       hand="$(arg hand)"
                       ee_id="$(arg ee_id)"

Commit message: stabilized arm prefix handling

File: robots/common/franka_arm.ros2_control.xacro (robot description, xacro)
@@ -12,5 +12,6 @@
                  gazebo_effort:=false
                  arm_prefix:=''">
-    <xacro:property name="arm_prefix_modified" value="${'' if arm_prefix == '' else arm_prefix + '_'}" />
+    <xacro:property name="arm_prefix_clean" value="${arm_prefix.rstrip('_')}" />
+    <xacro:property name="arm_prefix_modified" value="${'' if arm_prefix_clean == '' else arm_prefix_clean + '_'}" />
     <ros2_control name="${arm_prefix_modified}FrankaHardwareInterface" type="system">
         <hardware>
@@ -70,13 +71,13 @@
         </joint>
       </xacro:macro>
-      <xacro:configure_joint joint_name="${arm_prefix}${arm_id}_joint1" initial_position="0.0"/>
-      <xacro:configure_joint joint_name="${arm_prefix}${arm_id}_joint2" initial_position="${-pi/4}"/>
-      <xacro:configure_joint joint_name="${arm_prefix}${arm_id}_joint3" initial_position="0.0"/>
-      <xacro:configure_joint joint_name="${arm_prefix}${arm_id}_joint4" initial_position="${-3*pi/4}"/>
-      <xacro:configure_joint joint_name="${arm_prefix}${arm_id}_joint5" initial_position="0.0"/>
-      <xacro:configure_joint joint_name="${arm_prefix}${arm_id}_joint6" initial_position="${pi/2}"/>
-      <xacro:configure_joint joint_name="${arm_prefix}${arm_id}_joint7" initial_position="${pi/4}"/>
+      <xacro:configure_joint joint_name="${arm_prefix_modified}${arm_id}_joint1" initial_position="0.0"/>
+      <xacro:configure_joint joint_name="${arm_prefix_modified}${arm_id}_joint2" initial_position="${-pi/4}"/>
+      <xacro:configure_joint joint_name="${arm_prefix_modified}${arm_id}_joint3" initial_position="0.0"/>
+      <xacro:configure_joint joint_name="${arm_prefix_modified}${arm_id}_joint4" initial_position="${-3*pi/4}"/>
+      <xacro:configure_joint joint_name="${arm_prefix_modified}${arm_id}_joint5" initial_position="0.0"/>
+      <xacro:configure_joint joint_name="${arm_prefix_modified}${arm_id}_joint6" initial_position="${pi/2}"/>
+      <xacro:configure_joint joint_name="${arm_prefix_modified}${arm_id}_joint7" initial_position="${pi/4}"/>
       <xacro:if value="${gazebo and hand}">
-        <xacro:configure_joint joint_name="${arm_id}_finger_joint1" initial_position="0.0" />
+        <xacro:configure_joint joint_name="${arm_prefix_modified}${arm_id}_finger_joint1" initial_position="0.0" />
       </xacro:if>
       <xacro:unless value="${isaac}">
