Commit message: added environment for franka

File: robots/common/utils.xacro (robot description, xacro)
@@ -104,4 +104,19 @@
     </collision>
   </xacro:macro>
+  <!-- Added from original humation file: -->
+  <xacro:macro name="collision_rectangle" params="size:='0 0 0' xyz:='0 0 0' direction:='z'">
+    <xacro:property name="roll" value="${pi/2.0 if 'y' in direction else 0}" />
+    <xacro:property name="pitch" value="${pi/2.0 if 'x' in direction else 0}" />
+    <xacro:property name="yaw" value="0" />
+    <xacro:property name="x" value="${xyz.split(' ')[0]}" />
+    <xacro:property name="y" value="${xyz.split(' ')[1]}" />
+    <xacro:property name="z" value="${xyz.split(' ')[2]}" />
+    <collision>
+      <origin xyz="${x} ${y} ${z}" rpy="${roll} ${pitch} ${yaw}"/>
+      <geometry>
+        <box size="${size}" />
+      </geometry>
+    </collision>
+  </xacro:macro>
   <!-- ========================================================== -->
   <!-- Adds the required tags to simulate one joint in gazebo     -->

File: robots/fr3/fr3.urdf.xacro (robot description, xacro)
@@ -23,9 +23,12 @@
   <xacro:arg name="rpy_ee" default= "0 0 ${-pi/4}" />
   <!-- Position offset between ee frame and tcp frame -->
-  <xacro:arg name="tcp_xyz" default="0 0 0.1034" />
+  <!-- default was 0 0 0.1034, but this was changed in the original humation package so I adjusted it. -->
+  <xacro:arg name="tcp_xyz" default="0 0 0.0934" />
   <!-- Rotation offset between ee frame and tcp frame -->
   <xacro:arg name="tcp_rpy" default="0 0 0" />
   <!-- Safety distance for the collision capsules -->
-  <xacro:arg name="safety_distance" default="0.03" />
+  <!-- originally this was 0.03! (Changed because the original humation package had this value) -->
+  <!-- TODO: If something goes wrong: The original humation package also defined a seperate safety_distance for the end effector that was ignored here! -->
+  <xacro:arg name="safety_distance" default="0.02" />
   <!-- Should self-collision be enabled? -->
   <xacro:arg name="with_sc" default="false" />
@@ -78,3 +81,5 @@
                       connected_to= "base">
   </xacro:franka_robot>
+  <!-- Humation environment! -->
+  <xacro:include filename="$(find franka_description)/environment/environment.urdf"/>
 </robot>
