Commit message: remove arm_id to fix bug of fr3_fr3_ naming in franka

File: robots/common/franka_arm.srdf.xacro (robot description, xacro)
@@ -2,5 +2,6 @@
 <robot xmlns:xacro="http://www.ros.org/wiki/xacro" >
     <xacro:macro name="franka_arm_srdf" params="arm_id hand:='true' ee_id:=franka_hand arm_prefix='' no_prefix='false'">
-        <xacro:property name="prefix" value="${'' if no_prefix else arm_prefix + arm_id + '_'}" />
+        <!-- <xacro:property name="prefix" value="${'' if no_prefix else arm_prefix + arm_id + '_'}" /> -->
+        <xacro:property name="prefix" value="${'' if no_prefix else arm_prefix}" />
         <xacro:include filename="$(find franka_description)/robots/common/group_definition.xacro"/>
         <xacro:group_definition prefix="${prefix}" group_name="${prefix}arm" tip_link="${prefix}link8"/>
