Commit message: updated URDF to fit the new link names, fixed CMakeLists so that environment is installed.

File: environment/environment.urdf (robot description, URDF)
Before this commit: robot environment, 1 links, 1 joints
Joints:
- joint world_environment_joint: parent fr3_link0 -> franka_fr3_link0
